Commit message: Switch to Shoulder Sensor

File: urdf/ros2_control.xacro (robot description, xacro)
@@ -7,4 +7,5 @@
             <hardware>
                 <plugin>ros2_roamadome/RoamadomeControl</plugin>
+                <param name="serial_port">/dev/ttyACM0</param>
             </hardware>
             <joint name="dome_joint">
@@ -18,22 +19,22 @@
             <hardware>
                 <plugin>ros2_shoulder_sensor/MagneticAngleSensor</plugin>
-                <param name="static_position">0.5</param>
+                <param name="can_interface">can0</param>
+                <param name="stale_timeout_ms">200</param>
+                <param name="startup_timeout_ms">1000</param>
             </hardware>
-                <!-- optional hardware-level default -->
-                <joint name="left_shoulder_joint">
-                    <param name="static_position">-0.6283</param>
-                    <param name="invert_position">true</param>
-                </joint>
-                <joint name="right_shoulder_joint">
-                    <param name="static_position">0.6283</param>
-                </joint>
-                <!--
-                <joint name="left_ankle_joint">
-                    <param name="static_position">-0.31415</param>
-                </joint>
-                <joint name="right_ankle_joint">
-                    <param name="static_position">-0.31415</param>
-                </joint>
-                -->
+            <joint name="left_shoulder_joint">
+                <state_interface name="position"/>
+                <state_interface name="temperature"/>
+                <param name="node_id">3</param>
+                <param name="invert_position">false</param>
+                <param name="zero_offset_deg">0.0</param>
+            </joint>
+            <joint name="right_shoulder_joint">
+                <state_interface name="position"/>
+                <state_interface name="temperature"/>
+                <param name="node_id">4</param>
+                <param name="invert_position">false</param>
+                <param name="zero_offset_deg">1.5</param>
+            </joint>
         </ros2_control>
     <!--

Commit message: Adding ODrive Support

File: urdf/ros2_control.xacro (robot description, xacro)
@@ -3,4 +3,16 @@
     <xacro:unless value="$(arg sim_mode)">
         <ros2_control name="RealRobot" type="generic_system">
+        </ros2_control>
+        <ros2_control name="ODriveInterface" type="system">
+            <hardware>
+                <plugin>odrive_ros2_control_plugin/ODriveHardwareInterface</plugin>
+                <param name="can">can1</param>
+            </hardware>
+            <joint name="left_wheel_joint">
+                <param name="node_id">1</param>
+            </joint>
+            <joint name="right_wheel_joint">
+                <param name="node_id">2</param>
+            </joint>
         </ros2_control>
         <ros2_control name="RoamADome" type="actuator">

Commit message: Adding updates to support gear train of drive motors.

File: urdf/ros2_control.xacro (robot description, xacro)
@@ -15,4 +15,18 @@
                 <param name="node_id">2</param>
             </joint>
+            <transmission name="left_wheel_trans">
+                <plugin>transmission_interface/SimpleTransmission</plugin>
+                <actuator name="left_wheel_motor" role="actuator1"/>
+                <joint name="left_wheel_joint" role="joint1">
+                    <mechanical_reduction>12.6</mechanical_reduction>
+                </joint>
+            </transmission>
+            <transmission name="right_wheel_trans">
+                <plugin>transmission_interface/SimpleTransmission</plugin>
+                <actuator name="right_wheel_motor" role="actuator1"/>
+                <joint name="right_wheel_joint" role="joint1">
+                    <mechanical_reduction>12.6</mechanical_reduction>
+                </joint>
+            </transmission>
         </ros2_control>
         <ros2_control name="RoamADome" type="actuator">
@@ -38,5 +52,6 @@
                 <state_interface name="position"/>
                 <state_interface name="temperature"/>
-                <param name="node_id">3</param>
+                <!--<param name="node_id">3</param>-->
+                <param name="node_id">1</param>
                 <param name="invert_position">false</param>
                 <param name="zero_offset_deg">0.0</param>
@@ -45,5 +60,6 @@
                 <state_interface name="position"/>
                 <state_interface name="temperature"/>
-                <param name="node_id">4</param>
+                <!--<param name="node_id">4</param>-->
+                <param name="node_id">2</param>
                 <param name="invert_position">false</param>
                 <param name="zero_offset_deg">1.5</param>

Commit message: Updates to bring in a number of updates

File: urdf/ros2_control.xacro (robot description, xacro)
@@ -15,18 +15,4 @@
                 <param name="node_id">2</param>
             </joint>
-            <transmission name="left_wheel_trans">
-                <plugin>transmission_interface/SimpleTransmission</plugin>
-                <actuator name="left_wheel_motor" role="actuator1"/>
-                <joint name="left_wheel_joint" role="joint1">
-                    <mechanical_reduction>12.6</mechanical_reduction>
-                </joint>
-            </transmission>
-            <transmission name="right_wheel_trans">
-                <plugin>transmission_interface/SimpleTransmission</plugin>
-                <actuator name="right_wheel_motor" role="actuator1"/>
-                <joint name="right_wheel_joint" role="joint1">
-                    <mechanical_reduction>12.6</mechanical_reduction>
-                </joint>
-            </transmission>
         </ros2_control>
         <ros2_control name="RoamADome" type="actuator">
@@ -52,5 +38,5 @@
                 <state_interface name="position"/>
                 <state_interface name="temperature"/>
-                <!--<param name="node_id">3</param>-->
+                <!--param name="unique_id">df643cf0134b1a350000000000000000</param-->
                 <param name="node_id">1</param>
                 <param name="invert_position">false</param>
@@ -60,5 +46,5 @@
                 <state_interface name="position"/>
                 <state_interface name="temperature"/>
-                <!--<param name="node_id">4</param>-->
+                <!--param name="unique_id">df643cf013252b370000000000000000</param-->
                 <param name="node_id">2</param>
                 <param name="invert_position">false</param>
@@ -66,34 +52,4 @@
             </joint>
         </ros2_control>
-    <!--
-        <ros2_control name="RealRobot" type="system">
-            <hardware>
-                <plugin>diffdrive_arduino/DiffDriveArduinoHardware</plugin>
-                <param name="left_wheel_name">left_wheel_joint</param>
-                <param name="right_wheel_name">right_wheel_joint</param>
-                <param name="loop_rate">30</param>
-                <param name="device">/dev/ttyUSB0</param>
-                <param name="baud_rate">57600</param>
-                <param name="timeout_ms">1000</param>
-                <param name="enc_counts_per_rev">3436</param>
-            </hardware>
-            <joint name="left_wheel_joint">
-                <command_interface name="velocity">
-                    <param name="min">-10</param>
-                    <param name="max">10</param>
-                </command_interface>
-                <state_interface name="position"/>
-                <state_interface name="velocity"/>
-            </joint>
-            <joint name="right_wheel_joint">
-                <command_interface name="velocity">
-                    <param name="min">-10</param>
-                    <param name="max">10</param>
-                </command_interface>
-                <state_interface name="position"/>
-                <state_interface name="velocity"/>
-            </joint>
-        </ros2_control>
-        -->
     </xacro:unless>
 </robot>
