Commit message: Real Hardware Integration (#1)
* Switch to Shoulder Sensor

* Adding ODrive Support

* Adding updates to support gear train of drive motors.

* Updates to bring in a number of updates

* Fix verison typo to version in r2d2.repos for r2_sim and ros_odrive entries

Agent-Logs-Url: https://github.com/daveismith/r2_bringup/sessions/2c4f7928-538d-4ba4-aa77-d4fb2967ee06

Co-authored-by: daveismith <1734595+daveismith@users.noreply.github.com>

* Fixing issues raised by PR

* Switch  to serial number based port definition for the roam a dome.

---------

Co-authored-by: copilot-swe-agent[bot] <198982749+Copilot@users.noreply.github.com>

File: urdf/ros2_control.xacro (robot description, xacro)
@@ -2,9 +2,27 @@
 <robot xmlns:xacro="http://www.ros.org/wiki/xacro">
     <xacro:unless value="$(arg sim_mode)">
-        <ros2_control name="RealRobot" type="generic_system">
+        <ros2_control name="ODriveInterface" type="system">
+            <hardware>
+                <plugin>odrive_ros2_control_plugin/ODriveHardwareInterface</plugin>
+                <param name="can">can1</param>
+            </hardware>
+            <joint name="left_wheel_joint">
+                <command_interface name="velocity" />
+                <state_interface name="position" />
+                <state_interface name="velocity" />
+                <param name="node_id">1</param>
+            </joint>
+            <joint name="right_wheel_joint">
+                <command_interface name="velocity" />
+                <state_interface name="position" />
+                <state_interface name="velocity" />
+                <param name="node_id">2</param>
+            </joint>
         </ros2_control>
         <ros2_control name="RoamADome" type="actuator">
             <hardware>
                 <plugin>ros2_roamadome/RoamadomeControl</plugin>
+                <!--<param name="serial_port">/dev/ttyACM0</param>-->
+                <param name="serial_port">/dev/serial/by-id/usb-Espressif_USB_JTAG_serial_debug_unit_34:85:18:8B:35:34-if00</param>
             </hardware>
             <joint name="dome_joint">
@@ -18,53 +36,25 @@
             <hardware>
                 <plugin>ros2_shoulder_sensor/MagneticAngleSensor</plugin>
-                <param name="static_position">0.5</param>
+                <param name="can_interface">can0</param>
+                <param name="stale_timeout_ms">200</param>
+                <param name="startup_timeout_ms">1000</param>
             </hardware>
-                <!-- optional hardware-level default -->
-                <joint name="left_shoulder_joint">
-                    <param name="static_position">-0.6283</param>
-                    <param name="invert_position">true</param>
-                </joint>
-                <joint name="right_shoulder_joint">
-                    <param name="static_position">0.6283</param>
-                </joint>
-                <!--
-                <joint name="left_ankle_joint">
-                    <param name="static_position">-0.31415</param>
-                </joint>
-                <joint name="right_ankle_joint">
-                    <param name="static_position">-0.31415</param>
-                </joint>
-                -->
-        </ros2_control>
-    <!--
-        <ros2_control name="RealRobot" type="system">
-            <hardware>
-                <plugin>diffdrive_arduino/DiffDriveArduinoHardware</plugin>
-                <param name="left_wheel_name">left_wheel_joint</param>
-                <param name="right_wheel_name">right_wheel_joint</param>
-                <param name="loop_rate">30</param>
-                <param name="device">/dev/ttyUSB0</param>
-                <param name="baud_rate">57600</param>
-                <param name="timeout_ms">1000</param>
-                <param name="enc_counts_per_rev">3436</param>
-            </hardware>
-            <joint name="left_wheel_joint">
-                <command_interface name="velocity">
-                    <param name="min">-10</param>
-                    <param name="max">10</param>
-                </command_interface>
+            <joint name="left_shoulder_joint">
                 <state_interface name="position"/>
-                <state_interface name="velocity"/>
+                <state_interface name="temperature"/>
+                <!--param name="unique_id">df643cf0134b1a350000000000000000</param-->
+                <param name="node_id">1</param>
+                <param name="invert_position">false</param>
+                <param name="zero_offset_deg">0.0</param>
             </joint>
-            <joint name="right_wheel_joint">
-                <command_interface name="velocity">
-                    <param name="min">-10</param>
-                    <param name="max">10</param>
-                </command_interface>
+            <joint name="right_shoulder_joint">
                 <state_interface name="position"/>
-                <state_interface name="velocity"/>
+                <state_interface name="temperature"/>
+                <!--param name="unique_id">df643cf013252b370000000000000000</param-->
+                <param name="node_id">2</param>
+                <param name="invert_position">false</param>
+                <param name="zero_offset_deg">1.5</param>
             </joint>
         </ros2_control>
-        -->
     </xacro:unless>
 </robot>
